File: pcb-design/schematic.sch (KiCad schematic (older format))
At the start: 16 parts, among them J4 Screw_Terminal_01x02, J6 Conn_02x13_Top_Bottom, Q1 2N2222, Q2 2N2222, Q3 2N2222, Q6 2N2222, Q8 2N3906, U3 MCP2562-E-P, U4 AP1117-33, U6 ESP32-DEVKITC-32D

Commit message: Final changes for Rev 1 board, ordered 10/06/2020
Parts:
- added U7: L7805, Package_SIP:SIP3_11.6x8.5mm, symbol Regulator_Linear:L7805
- U4: footprint Package_TO_SOT_SMD:SOT-223-3_TabPin2 -> Package_SIP:SIP3_11.6x8.5mm
Connections:
- net +12V: now also U7.1 (IN)
- net +5V: now also U7.3 (OUT)
- net A0_SourceOutput: now also J6.21 (Pin_21); no longer J6.1 (Pin_1)
- net A1_SourceOutput: now also J6.20 (Pin_20); no longer J6.2 (Pin_2)
- net A2_SourceOutput: now also J6.19 (Pin_19); no longer J6.3 (Pin_3)
- net A3_SourceOutput: now also J6.18 (Pin_18); no longer J6.4 (Pin_4)
- net A4_SourceOutput: now also J6.17 (Pin_17); no longer J6.5 (Pin_5)
- net A5_SourceOutput: now also J6.16 (Pin_16); no longer J6.6 (Pin_6)
- net A6_SourceOutput: now also J6.15 (Pin_15); no longer J6.7 (Pin_7)
- net A7_SourceOutput: now also J6.14 (Pin_14); no longer J6.8 (Pin_8)
- net B0_SinkOutput: now also J6.1 (Pin_1); no longer J6.14 (Pin_14)
- net B1_SinkOutput: now also J6.2 (Pin_2); no longer J6.15 (Pin_15)
- net B2_SinkOutput: now also J6.3 (Pin_3); no longer J6.16 (Pin_16)
- net B3_SinkOutput: now also J6.4 (Pin_4); no longer J6.17 (Pin_17)
- net B4_SinkOutput: now also J6.5 (Pin_5); no longer J6.18 (Pin_18)
- net B5_SinkOutput: now also J6.6 (Pin_6); no longer J6.19 (Pin_19)
- net B6_SinkOutput: now also J6.7 (Pin_7); no longer J6.20 (Pin_20)
- net B7_SinkOutput: now also J6.8 (Pin_8); no longer J6.21 (Pin_21)
- net FuelGauge: now also J6.23 (Pin_23); no longer J6.25 (Pin_25)
- net GND: now also U7.2 (GND)
- net Speedometer: now also J6.24 (Pin_24); no longer J6.23 (Pin_23)
- net Tachometer: now also J6.22 (Pin_22); no longer J6.24 (Pin_24)
- net TempGauge: now also J6.25 (Pin_25); no longer J6.22 (Pin_22)
Other:
- note added: "5v Power Supply"
Changed lines of the file:
@@
 F 0 "U4" H 5050 2542 50  0000 C CNN
 F 1 "AP1117-33" H 5050 2451 50  0000 C CNN
-F 2 "Package_TO_SOT_SMD:SOT-223-3_TabPin2" H 5050 2500 50  0001 C CNN
+F 2 "Package_SIP:SIP3_11.6x8.5mm" H 5050 2500 50  0001 C CNN
 F 3 "http://www.diodes.com/datasheets/AP1117.pdf" H 5150 2050 50  0001 C CNN
 	1    5050 2300
@@
 Text GLabel 7500 4850 2    50   Input ~ 0
 A7_SourceOutput
+Text GLabel 9550 4900 2    50   Input ~ 0
+A0_SourceOutput
+Text GLabel 9550 4800 2    50   Input ~ 0
+A1_SourceOutput
+Text GLabel 9550 4700 2    50   Input ~ 0
+A2_SourceOutput
+Text GLabel 9550 4600 2    50   Input ~ 0
+A3_SourceOutput
+Text GLabel 9550 4500 2    50   Input ~ 0
+A4_SourceOutput
+Text GLabel 9550 4400 2    50   Input ~ 0
+A5_SourceOutput
+Text GLabel 9550 4300 2    50   Input ~ 0
+A6_SourceOutput
+Text GLabel 9550 4200 2    50   Input ~ 0
+A7_SourceOutput
 Text GLabel 9050 4200 0    50   Input ~ 0
-A0_SourceOutput
+B0_SinkOutput
 Text GLabel 9050 4300 0    50   Input ~ 0
-A1_SourceOutput
+B1_SinkOutput
 Text GLabel 9050 4400 0    50   Input ~ 0
-A2_SourceOutput
+B2_SinkOutput
 Text GLabel 9050 4500 0    50   Input ~ 0
-A3_SourceOutput
+B3_SinkOutput
 Text GLabel 9050 4600 0    50   Input ~ 0
-A4_SourceOutput
+B4_SinkOutput
 Text GLabel 9050 4700 0    50   Input ~ 0
-A5_SourceOutput
+B5_SinkOutput
 Text GLabel 9050 4800 0    50   Input ~ 0
-A6_SourceOutput
+B6_SinkOutput
 Text GLabel 9050 4900 0    50   Input ~ 0
-A7_SourceOutput
-Text GLabel 9550 4200 2    50   Input ~ 0
-B0_SinkOutput
-Text GLabel 9550 4300 2    50   Input ~ 0
-B1_SinkOutput
-Text GLabel 9550 4400 2    50   Input ~ 0
-B2_SinkOutput
-Text GLabel 9550 4500 2    50   Input ~ 0
-B3_SinkOutput
-Text GLabel 9550 4600 2    50   Input ~ 0
-B4_SinkOutput
-Text GLabel 9550 4700 2    50   Input ~ 0
-B5_SinkOutput
-Text GLabel 9550 4800 2    50   Input ~ 0
-B6_SinkOutput
-Text GLabel 9550 4900 2    50   Input ~ 0
 B7_SinkOutput
 Wire Notes Line
@@
 	1    0    0    -1
 $EndComp
+Text GLabel 9550 5300 2    50   Input ~ 0
+TempGauge
+Text GLabel 9550 5100 2    50   Input ~ 0
+FuelGauge
+Text GLabel 9550 5200 2    50   Input ~ 0
+Speedometer
 Text GLabel 9550 5000 2    50   Input ~ 0
-TempGauge
-Text GLabel 9550 5300 2    50   Input ~ 0
-FuelGauge
-Text GLabel 9550 5100 2    50   Input ~ 0
-Speedometer
-Text GLabel 9550 5200 2    50   Input ~ 0
 Tachometer
 $Comp
@@
 	0    1    1    0
 $EndComp
+$Comp
+L Regulator_Linear:L7805 U7
+U 1 1 5EE03F14
+P 4850 3300
+F 0 "U7" H 4850 3542 50  0000 C CNN
+F 1 "L7805" H 4850 3451 50  0000 C CNN
+F 2 "Package_SIP:SIP3_11.6x8.5mm" H 4875 3150 50  0001 L CIN
+F 3 "http://www.st.com/content/ccc/resource/technical/document/datasheet/41/4f/b3/b0/12/d4/47/88/CD00000444.pdf/files/CD00000444.pdf/jcr:content/translations/en.CD00000444.pdf" H 4850 3250 50  0001 C CNN
+	1    4850 3300
+	1    0    0    -1
+$EndComp
+$Comp
+L power:GND #PWR0148
+U 1 1 5EE0400D
+P 4850 3600
+F 0 "#PWR0148" H 4850 3350 50  0001 C CNN
+F 1 "GND" H 4855 3427 50  0000 C CNN
+F 2 "" H 4850 3600 50  0001 C CNN
+F 3 "" H 4850 3600 50  0001 C CNN
+	1    4850 3600
+	1    0    0    -1
+$EndComp
+$Comp
+L power:+12V #PWR0149
+U 1 1 5EE04058
+P 4550 3300
+F 0 "#PWR0149" H 4550 3150 50  0001 C CNN
+F 1 "+12V" H 4565 3473 50  0000 C CNN
+F 2 "" H 4550 3300 50  0001 C CNN
+F 3 "" H 4550 3300 50  0001 C CNN
+	1    4550 3300
+	1    0    0    -1
+$EndComp
+$Comp
+L power:+5V #PWR0150
+U 1 1 5EE040A3
+P 5150 3300
+F 0 "#PWR0150" H 5150 3150 50  0001 C CNN
+F 1 "+5V" H 5165 3473 50  0000 C CNN
+F 2 "" H 5150 3300 50  0001 C CNN
+F 3 "" H 5150 3300 50  0001 C CNN
+	1    5150 3300
+	1    0    0    -1
+$EndComp
+Text Notes 4150 3000 0    50   ~ 0
+5v Power Supply
+Wire Notes Line
+	4100 2900 5600 2900
+Wire Notes Line
+	5600 2900 5600 3850
+Wire Notes Line
+	5600 3850 4100 3850
+Wire Notes Line
+	4100 3850 4100 2900
 $EndSCHEMATC
