File: pcb-design/schematic.sch (KiCad schematic (older format))
At the start: 17 parts, among them J4 Screw_Terminal_01x02, J6 Conn_02x13_Top_Bottom, Q1 2N2222, Q2 2N2222, Q3 2N2222, Q6 2N2222, Q8 2N3906, U3 MCP2562-E-P, U4 AP1117-33, U6 ESP32-DEVKITC-32D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

Commit message: Updated resistor footprints to 0805 which had better coverage for JLCPCB basic parts.
Parts:
- R1, R2, R3, R9: footprint Resistor_SMD:R_1206_3216Metric_Pad1.42x1.75mm_HandSolder -> Resistor_SMD:R_0805_2012Metric
- R10, R7: value 4000 -> 4700; footprint Resistor_SMD:R_1206_3216Metric_Pad1.42x1.75mm_HandSolder -> Resistor_SMD:R_0805_2012Metric
Changed lines of the file:
@@
 F 0 "R2" V 9095 3300 50  0000 C CNN
 F 1 "220" V 9186 3300 50  0000 C CNN
-F 2 "Resistor_SMD:R_1206_3216Metric_Pad1.42x1.75mm_HandSolder" H 9300 3300 50  0001 C CNN
+F 2 "Resistor_SMD:R_0805_2012Metric" H 9300 3300 50  0001 C CNN
 F 3 "~" H 9300 3300 50  0001 C CNN
 	1    9300 3300
@@
 F 0 "R1" V 9095 2400 50  0000 C CNN
 F 1 "470" V 9186 2400 50  0000 C CNN
-F 2 "Resistor_SMD:R_1206_3216Metric_Pad1.42x1.75mm_HandSolder" H 9300 2400 50  0001 C CNN
+F 2 "Resistor_SMD:R_0805_2012Metric" H 9300 2400 50  0001 C CNN
 F 3 "~" H 9300 2400 50  0001 C CNN
 	1    9300 2400
@@
 F 0 "R3" V 6745 2400 50  0000 C CNN
 F 1 "470" V 6836 2400 50  0000 C CNN
-F 2 "Resistor_SMD:R_1206_3216Metric_Pad1.42x1.75mm_HandSolder" H 6950 2400 50  0001 C CNN
+F 2 "Resistor_SMD:R_0805_2012Metric" H 6950 2400 50  0001 C CNN
 F 3 "~" H 6950 2400 50  0001 C CNN
 	1    6950 2400
@@
 AR Path="/5E6B979D/5E6C4604" Ref="R?"  Part="1"
 F 0 "R10" V 8395 1200 50  0000 C CNN
-F 1 "4000" V 8486 1200 50  0000 C CNN
-F 2 "Resistor_SMD:R_1206_3216Metric_Pad1.42x1.75mm_HandSolder" H 8600 1200 50  0001 C CNN
+F 1 "4700" V 8486 1200 50  0000 C CNN
+F 2 "Resistor_SMD:R_0805_2012Metric" H 8600 1200 50  0001 C CNN
 F 3 "~" H 8600 1200 50  0001 C CNN
 	1    8600 1200
@@
 F 0 "R9" V 8395 900 50  0000 C CNN
 F 1 "22000" V 8486 900 50  0000 C CNN
-F 2 "Resistor_SMD:R_1206_3216Metric_Pad1.42x1.75mm_HandSolder" H 8600 900 50  0001 C CNN
+F 2 "Resistor_SMD:R_0805_2012Metric" H 8600 900 50  0001 C CNN
 F 3 "~" H 8600 900 50  0001 C CNN
 	1    8600 900
@@
 AR Path="/5E6B979D/5E6C4617" Ref="R?"  Part="1"
 F 0 "R7" V 7845 1450 50  0000 C CNN
-F 1 "4000" V 7936 1450 50  0000 C CNN
-F 2 "Resistor_SMD:R_1206_3216Metric_Pad1.42x1.75mm_HandSolder" H 8050 1450 50  0001 C CNN
+F 1 "4700" V 7936 1450 50  0000 C CNN
+F 2 "Resistor_SMD:R_0805_2012Metric" H 8050 1450 50  0001 C CNN
 F 3 "~" H 8050 1450 50  0001 C CNN
 	1    8050 1450
