File: pcb-design/schematic.sch (KiCad schematic (older format))
At the start: 16 parts, among them J1 TempGauge, J2 FuelGauge, J3 SpeedInput_C2_P10-13, Q1 2N2222, Q2 2N2222, Q3 2N2222, Q4 2N3906, Q5 2N2222

Commit message: Squashed commit of the following:
commit 3feebbdd7fc9a19dcfe87aea05ec82215f171dbb
Author: dowster <brady@dowster.net>
Date:   Mon Feb 13 23:49:32 2023 -0600

    add potential backup MCU

commit 7657e025624eaa3ad175eda664276684d823e8da
Author: dowster <brady@dowster.net>
Date:   Sun Jun 14 00:02:21 2020 -0500

    Revert "Trying to add a pdf of the pcb layout"

    This reverts commit b56f1969f75d8c114cc69d4ada7bfdc8b18707b8.

commit 2fa9ff3b8e4192675af680a6f10c74fef6b1e3eb
Author: dowster <brady@dowster.net>
Date:   Sun Jun 14 00:00:47 2020 -0500

    Trying to add a pdf of the pcb layout

commit dd21b1a7d9b37009cc4babccdf1aa4f396be8d7d
Author: dowster <brady@dowster.net>
Date:   Sat Jun 13 23:53:15 2020 -0500

    Updated resistor footprints to 0805 which had better coverage for JLCPCB basic parts.

commit 8307c3e4bc4598d6275d93f7cccdc8af7ce4bc90
Author: dowster <brady@dowster.net>
Date:   Wed Jun 10 00:56:32 2020 -0500

    Final changes for Rev 1 board, ordered 10/06/2020

commit 434b86fbaa718e58593fb08e1f55d7f9f253070a
Author: dowster <brady@dowster.net>
Date:   Tue Jun 9 02:26:57 2020 -0500

    Added TE 827881-1 connector and footprint
    re-arranged schematic

commit 6d09ca954eead60ab9723ebacf2d3cc768a60194
Author: dowster <brady@dowster.net>
Date:   Tue Jun 9 00:57:00 2020 -0500

    checkin

commit c2e850715b8f67c56e717ab6a99da3764dfebaa0
Author: dowster <brady@dowster.net>
Date:   Tue May 5 01:29:08 2020 -0500

    Swapped the esp32 symbol and footprint to be one for the dev modules so I can just populate the boards with standoffs.

    Wired up some more nets and made the layout a little prettier.

commit ea3064ef9aa3745e3f10cc965f2b7b57569e8fb9
Author: dowster <brady@dowster.net>
Date:   Fri May 1 22:08:50 2020 -0500

    Moved some files around

commit 5fb95e82d58e494b6845b6b07395a5ce6095db6f
Author: dowster <brady@dowster.net>
Date:   Sun Mar 22 01:33:21 2020 -0500

    Checking in schematic files

commit 23cadce822c5ff0c7eff896b529663319354c8b2
Auth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
Parts:
- removed J1: TempGauge, symbol Connector:Conn_01x01_Male
- removed J2: FuelGauge, symbol Connector:Conn_01x01_Male
- removed J3, J?: SpeedInput_C2_P10-13, symbol Connector:Conn_01x01_Male
- removed Q4: 2N3906, Package_TO_SOT_THT:TO-92_Inline, symbol Transistor_BJT:2N3906
- removed Q5: 2N2222, symbol Device:Q_NPN_BCE
- removed R4, R6: 4000, symbol Device:R_Small_US
- removed R5: 22000, symbol Device:R_Small_US
- removed U?: ESP32-WROOM-32, RF_Module:ESP32-WROOM-32, symbol RF_Module:ESP32-WROOM-32
- added J4: Screw_Terminal_01x02, TerminalBlock_TE-Connectivity:TerminalBlock_TE_282834-2_1x02_P2.54mm_Horizontal, symbol Connector:Screw_Terminal_01x02
- added J6: Conn_02x13_Top_Bottom, pcb-design:Connector_TE_827881-1, symbol Connector_Generic:Conn_02x13_Top_Bottom
- added Q6: 2N2222, Package_TO_SOT_THT:TO-92_HandSolder, symbol Device:Q_NPN_BCE
- added Q8: 2N3906, Package_TO_SOT_THT:TO-92_Inline, symbol Transistor_BJT:2N3906
- added R10, R7: 4700, Resistor_SMD:R_0805_2012Metric, symbol Device:R_Small_US
- added R9: 22000, Resistor_SMD:R_0805_2012Metric, symbol Device:R_Small_US
- added U3: MCP2562-E-P, Package_DIP:DIP-8_W7.62mm, symbol Interface_CAN_LIN:MCP2562-E-P
- added U4: AP1117-33, Package_SIP:SIP3_11.6x8.5mm, symbol Regulator_Linear:AP1117-33
- added U6: ESP32-DEVKITC-32D, pcb-design:MODULE_ESP32-DEVKITC-32D, symbol ESP32-DEVKITC-32D:ESP32-DEVKITC-32D
- added U7: L7805, Package_SIP:SIP3_11.6x8.5mm, symbol Regulator_Linear:L7805
- Q1, Q2, Q3: footprint (none) -> Package_TO_SOT_THT:TO-92_HandSolder
- R1, R2, R3: footprint (none) -> Resistor_SMD:R_0805_2012Metric
Connections:
- net labels added: +3V3, +5V, A0_SourceOutput, A1_SourceOutput, A2_SourceOutput, A3_SourceOutput, A4_SourceOutput, A5_SourceOutput, A6_SourceOutput, A7_SourceOutput, B0_SinkOutput, B1_SinkOutput, B2_SinkOutput, B3_SinkOutput, B4_SinkOutput, B5_SinkOutput, B6_SinkOutput, B7_SinkOutput, CAN0_H, CAN0_L, ESP_CAN0_RX, ESP_CAN0_TX, FuelGauge, I2C0_SCK, I2C0_SDA, Speedometer, SpeedometerSignal, Tachometer, TempGauge
- net labels removed: SpeedometerOutput
- wire segments 6 -> 13
Other:
- note added: "3.3v Power Supply\n"
- note added: "5v Power Supply"
- note added: "CANBus Transciever"
- note added: "ESP32 MCU"
- note added: "Fuel Gauge \nTransistor\n"
- note added: "Indicator Light Subsystem"
- note added: "Primary Connector\n"
- note added: "Speedometer Output\nTransistor"
- note added: "Tachometer Output \nDarlington Transistor - +12v"
- note added: "Termperature Gauge\nTransistor\n"
- moved on the sheet: Q1, Q2, Q3, R1, R2, R3
