File: pcb-design/Indicator_Lights.sch (KiCad schematic (older format))
At the start: 57 parts, among them U2 MCP23017_SP

Commit message: Updated resistor footprints to 0805 which had better coverage for JLCPCB basic parts.
Parts:
- R_A0_1, R_A0_3, R_A1_1, R_A1_3, R_A2_1, R_A2_3, R_A3_1, R_A3_3, R_A4_1, R_A4_3, R_A5_1, R_A5_3, R_A6_1, R_A6_3, R_A7_1, R_A7_3, R_B0_1, R_B1_1, R_B2_1, R_B3_1, R_B4_1, R_B5_1, R_B6_1, R_B7_1: value 4000 -> 4700; footprint Resistor_SMD:R_1206_3216Metric_Pad1.42x1.75mm_HandSolder -> Resistor_SMD:R_0805_2012Metric
- R_A0_2, R_A1_2, R_A2_2, R_A3_2, R_A4_2, R_A5_2, R_A6_2, R_A7_2: footprint Resistor_SMD:R_1206_3216Metric_Pad1.42x1.75mm_HandSolder -> Resistor_SMD:R_0805_2012Metric
